File: Hardware/PCB/logic.kicad_sch (KiCad schematic)
At the start: 9 parts

Commit message: Finished schematic
Parts:
- removed AND4, AND6, AND8, OR1: 74HC04, symbol 74xx:74HC04
- removed AND5 (x2), AND6A1, AND6B1, AND9: 74HC08, symbol 74xx:74LS08
- removed OR2: 74LS32, symbol 74xx:74LS32
