File: Hardware/PCB/power.kicad_sch (KiCad schematic)
At the start: 8 parts, among them U1 74HC00, U2 74HC04, U3 74HC08, U5 74HC08, U6 74LS32, U7 74HC393, U8 74HC393

Commit message: Writing maybe working, also started on other parts of schematic
Parts:
- added U4: (no value), symbol custom:AT28C256
Connections:
- net +5V: now also U4.28 (Vcc)
- net GND: now also U4.14 (GND)
Changed lines of the file:
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@@
+	)
+	(junction
+		(at 181.61 57.15)
+		(diameter 0)
+		(color 0 0 0 0)
 	)
 	(junction
@@
 	)
 	(junction
+		(at 181.61 31.75)
+		(diameter 0)
+		(color 0 0 0 0)
+	)
+	(junction
 		(at 58.42 57.15)
 		(diameter 0)
@@
 	(wire
 		(pts
+			(xy 181.61 57.15) (xy 199.39 57.15)
+		)
+		(stroke
+			(width 0)
+			(type default)
+		)
+	)
+	(wire
+		(pts
 			(xy 78.74 57.15) (xy 99.06 57.15)
 		)
@@
 	(wire
 		(pts
+			(xy 199.39 57.15) (xy 199.39 55.88)
+		)
+		(stroke
+			(width 0)
+			(type default)
+		)
+	)
+	(wire
+		(pts
 			(xy 36.83 31.75) (xy 58.42 31.75)
 		)
@@
 	(wire
 		(pts
+			(xy 181.61 31.75) (xy 199.39 31.75)
+		)
+		(stroke
+			(width 0)
+			(type default)
+		)
+	)
+	(wire
+		(pts
 			(xy 36.83 57.15) (xy 58.42 57.15)
 		)
@@
 		(pts
 			(xy 58.42 57.15) (xy 78.74 57.15)
+		)
+		(stroke
+			(width 0)
+			(type default)
+		)
+	)
+	(wire
+		(pts
+			(xy 199.39 31.75) (xy 199.39 34.29)
 		)
 		(stroke
@@
 					(unit 1)
 				)
+			)
+		)
+	)
+	(symbol
+		(lib_id "custom:AT28C256")
+		(at 194.31 36.83 0)
+		(unit 1)
+		(body_style 1)
+		(exclude_from_sim no)
+		(in_bom yes)
+		(on_board yes)
+		(in_pos_files yes)
+		(dnp no)
+		(fields_autoplaced yes)
+		(property "Reference" "U4"
+			(at 205.74 45.0849 0)
+			(show_name no)
+			(do_not_autoplace no)
+			(effects
+				(font
+					(size 1.27 1.27)
+				)
+				(justify left)
+			)
+		)
+		(property "Value" ""
+			(at 194.31 36.83 0)
+			(show_name no)
+			(do_not_autoplace no)
+			(effects
+				(font
+					(size 1.27 1.27)
+				)
+			)
+		)
+		(property "Footprint" ""
+			(at 194.31 36.83 0)
+			(hide yes)
+			(show_name no)
+			(do_not_autoplace no)
+			(effects
+				(font
+					(size 1.27 1.27)
+				)
+			)
+		)
+		(property "Datasheet" ""
+			(at 194.31 36.83 0)
+			(hide yes)
+			(show_name no)
+			(do_not_autoplace no)
+			(effects
+				(font
+					(size 1.27 1.27)
+				)
+			)
+		)
+		(property "Description" ""
+			(at 194.31 36.83 0)
+			(hide yes)
+			(show_name no)
+			(do_not_autoplace no)
+			(effects
+				(font
+					(size 1.27 1.27)
+				)
+			)
+		)
+		(pin "5"
+		)
+		(pin "6"
+		)
+		(pin "22"
+		)
+		(pin "11"
+		)
+		(pin "13"
+		)
+		(pin "3"
+		)
+		(pin "4"
+		)
+		(pin "28"
+		)
+		(pin "23"
+		)
+		(pin "1"
+		)
+		(pin "16"
+		)
+		(pin "12"
+		)
+		(pin "19"
+		)
+		(pin "21"
+		)
+		(pin "26"
+		)
+		(pin "27"
+		)
+		(pin "10"
+		)
+		(pin "7"
+		)
+		(pin "14"
+		)
+		(pin "20"
+		)
+		(pin "2"
+		)
+		(pin "9"
+		)
+		(pin "15"
+		)
+		(pin "25"
+		)
+		(pin "24"
+		)
+		(pin "18"
+		)
+		(pin "17"
+		)
+		(pin "8"
+		)
+		(instances
+			(project "EEPROM-Programmer"
+				(path "/d87f1d9a-2aed-49cd-be27-2f3d60d4f0c5/1315f4d7-820d-4681-8246-98197c8ffaa8"
+					(reference "U4")
+					(unit 1)
+				)

Commit message: Finished schematic
Parts:
- added C10, C11, C12, C13, C14, C15, C16, C17, C3, C4, C5, C6, C7, C8, C9: C, symbol Device:C
- added U15: 74HC00, symbol 74xx:74HC00
Connections:
- net +5V: now also C10.1, C11.1, C12.1, C13.1, C14.1, C15.1, C16.1, C17.1, C3.1, C4.1, C5.1, C6.1, C7.1, C8.1, C9.1, U15.14 (VCC)
- net GND: now also C10.2, C11.2, C12.2, C13.2, C14.2, C15.2, C16.2, C17.2, C3.2, C4.2, C5.2, C6.2, C7.2, C8.2, C9.2, U15.7 (GND)
Other:
- note added: "Decoupling Capacitors"
