File: Hardware/PCB/stateMachine.kicad_sch (KiCad schematic)
At the start: 18 parts, among them U7 74HC393, U8 74HC393

Commit message: Finished schematic
Parts:
- added unit 1 of AND1
- added AND4, AND5, AND6A1, AND6B1, AND7, AND8, ANDb1: 74HC08, symbol 74xx:74LS08
- added AND6, NOT1, NOT2: 74HC04, symbol 74xx:74HC04
- added D4: Activity LED, symbol Device:LED
- added R4: R, symbol Device:R
- added U15: 74HC00, symbol 74xx:74HC00
Connections:
- net GND: now also AND1.1, AND1.2, ANDb1.4, ANDb1.5, D4.1 (K), U15.4, U15.5
- net State lsb: now also AND5.9, AND6.11
- net State msb: now also AND5.10, AND6B1.12
- net Secondary Clock: now reaches AND1.6, U7.1 (CP)
- net Secondary Clock: now also AND7.13
- net Bit Counter Not 0 renamed Bit Counter Not Zero
- net Bit Counter Not Zero: now also AND4.13, AND8.5
- net End Byte renamed UART Stop bit
- net UART Stop bit: now also AND4.3, AND6B1.13
- net UART Start Bit renamed Set UART Activity
- new net: AND4.12, AND4.4
- new net: AND6.10, AND6A1.9
- new net: AND8.4, AND8.6
- new net: D4.2 (A), R4.2
- new net: U15.12, U15.13, U15.3
- new net: AND6A1.10, AND6B1.11
- new net Command Finished: AND6A1.8
- new net EEPROM Output Enable: NOT2.8, U15.9
- new net EEPROM Write Enable: U15.8
- new net Is Sending: AND5.8, AND8.5, U15.2
- new net R~{W} EEPROM: NOT2.9, R4.1
- new net Sending Uart Data bits-time: U15.10, U15.11
- new net Shift In Clock: AND7.11
- new net Start Sending: AND8.6, NOT1.13
- new net UART Data bits-time: AND4.11, AND7.12
- new net ~{Start Sending}: NOT1.12, U15.1
- no-connect marks 15 -> 18
Other:
- note added: "Also redundant, should be able to use UART Data bit-time instead."
- note added: "Gate is redundant. Could use Primary Clock instead."
- note added: "The device cycles through four states, stored in Machine State. 0-2: The device is reciving or waiting for a byte a byte for each state. 3: Once the device recives 3 bytes, it then sends a byte. The behavior is the same for both reads and writes to the eeprom, resulting in a garbage byte being sent for either operation."
- note added: "UART Clock Divider"
- note added: "Unused Gates. Given the redundant gates elsewhere, it seems possible to reduce the chip count of this device. The goal is to get something that works, though, and this configuration is currently working on a breadboard."
- note removed: "Gate is redundant"
- note removed: "Timed Clock Divider"
- moved on the sheet: AND12C, AND1B, AND2A, AND3C, D1, D2, D3, JP1, JP2, OR3A1B, OR3B1C, OR3C1D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
